File: PureRingMod-panel.brd (EAGLE design)
At the start: 128.5 x 60.3 mm, 1 part

Commit message: Panel Design
Parts:
- flipped U$2 to the bottom, turned to 270 degrees
Other:
- board text added: "Modulator Volume"
Changed lines of the file:
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@@
 </layers>
 <board>
-<fusionsync huburn="a.cGVyc29uYWw6dWUyYjcyYjhk" projecturn="a.cGVyc29uYWw6dWUyYjcyYjhkIzIwMTgwMzMxMTI1NDI1ODAx" f3durn="urn:adsk.wipprod:dm.lineage:yTvX96VlTXqc7SVYm6EbHw" pcbguid="92f95855-f1de-4771-bb78-bd8b88de37d5" lastpulledtime="" lastsyncedchangeguid="93d8453b-91b8-59d5-a3a1-d16215728a67"/>
+<fusionsync huburn="a.cGVyc29uYWw6dWUyYjcyYjhk" projecturn="a.cGVyc29uYWw6dWUyYjcyYjhkIzIwMTgwMzMxMTI1NDI1ODAx" f3durn="urn:adsk.wipprod:dm.lineage:yTvX96VlTXqc7SVYm6EbHw" pcbguid="92f95855-f1de-4771-bb78-bd8b88de37d5" lastpulledtime="" lastsyncedchangeguid="3d2ef7b1-878d-d0ac-978d-303d17d2f0f3"/>
 <plain>
 <wire x1="-14.73" y1="-1.105" x2="113.77" y2="-1.105" width="0" layer="20"/>
@@
 <wire x1="113.77" y1="59.195" x2="-14.75" y2="59.195" width="0" layer="20"/>
 <wire x1="-14.75" y1="59.195" x2="-14.73" y2="-1.105" width="0" layer="20"/>
-<text x="101.6" y="2.54" size="1.016" layer="25" rot="R90">Ring Modulator
+<text x="91.44" y="20.32" size="1.016" layer="26" rot="SMR270">Ring Modulator
 Design Andy C
 From a design by Roman Sowa</text>
-<text x="109.22" y="2.54" size="1.016" layer="25" rot="R90">CC BY 3.0 </text>
-<text x="105.41" y="2.54" size="1.016" layer="25" rot="R90">V1.0</text>
+<text x="97.79" y="20.32" size="1.016" layer="26" rot="SMR270">CC BY 3.0 </text>
+<text x="93.98" y="20.32" size="1.016" layer="26" rot="SMR270">V1.0</text>
 <circle x="66.04" y="49.53" radius="3.162275" width="0.1524" layer="46"/>
 <circle x="11.43" y="49.53" radius="3.162275" width="0.1524" layer="46"/>
@@
 <circle x="66.04" y="27.94" radius="2.83980625" width="0.1524" layer="46"/>
 <circle x="30.48" y="7.62" radius="2.83980625" width="0.1524" layer="46"/>
-<text x="74.93" y="44.45" size="1.778" layer="25" font="fixed" ratio="9" rot="R90">Output 2</text>
-<text x="74.93" y="3.81" size="1.778" layer="25" font="fixed" ratio="9" rot="R90">Output</text>
+<text x="73.66" y="12.7" size="1.778" layer="26" font="fixed" ratio="9" rot="SMR270">Output 2</text>
+<text x="72.39" y="53.34" size="1.778" layer="26" font="fixed" ratio="9" rot="SMR270">Output</text>
 <circle x="21.59" y="27.94" radius="9.45" width="0.1524" layer="46"/>
-<text x="72.39" y="26.67" size="1.778" layer="25" font="fixed" ratio="9" rot="R90">Gain</text>
-<text x="53.34" y="26.67" size="1.778" layer="25" font="fixed" ratio="9" rot="R90">Mix</text>
-<text x="53.34" y="44.45" size="1.778" layer="25" font="fixed" ratio="9" rot="R90">Mic Mix</text>
-<text x="35.56" y="44.45" size="1.778" layer="25" font="fixed" ratio="9" rot="R90">Output 2</text>
-<text x="20.32" y="44.45" size="1.778" layer="25" font="fixed" ratio="9" rot="R90">Carrier</text>
-<text x="39.37" y="25.4" size="1.778" layer="25" font="fixed" ratio="9" rot="R90">Mic In</text>
-<text x="39.37" y="3.81" size="1.778" layer="25" font="fixed" ratio="9" rot="R90">Carrier
+<text x="72.39" y="30.48" size="1.778" layer="26" font="fixed" ratio="9" rot="SMR270">Gain</text>
+<text x="53.34" y="30.48" size="1.778" layer="26" font="fixed" ratio="9" rot="SMR270">Mix</text>
+<text x="53.34" y="53.34" size="1.778" layer="26" font="fixed" ratio="9" rot="SMR270">Mic Mix</text>
+<text x="40.64" y="13.97" size="1.778" layer="26" font="fixed" ratio="9" rot="SMR270">Modulator
 Volume</text>
-<text x="20.32" y="2.54" size="1.778" layer="25" font="fixed" ratio="9" rot="R90">Modulator</text>
-<text x="-5.08" y="16.51" size="2.54" layer="27" rot="R90">Pure Ring Modulator</text>
+<text x="20.32" y="54.61" size="1.778" layer="26" font="fixed" ratio="9" rot="SMR270">Carrier</text>
+<text x="36.83" y="33.02" size="1.778" layer="26" font="fixed" ratio="9" rot="SMR270">Mic In</text>
+<text x="39.37" y="54.61" size="1.778" layer="26" font="fixed" ratio="9" rot="SMR270">Carrier
+Volume</text>
+<text x="20.32" y="13.97" size="1.778" layer="26" font="fixed" ratio="9" rot="SMR270">Modulator</text>
+<text x="-5.08" y="46.99" size="2.54" layer="26" rot="SMR270">Pure Ring Modulator</text>
 </plain>
 <attributes>
@@
 </autorouter>
 <elements>
-<element name="U$2" library="gmsnLogo" package="GMSN!_LOGO" value="" x="0.23" y="30.95875" rot="R90"/>
+<element name="U$2" library="gmsnLogo" package="GMSN!_LOGO" value="" x="0.23" y="30.95875" rot="MR270"/>
 </elements>
 <signals>
