File: PureRingMod-panel.brd (EAGLE design)
At the start: 128.5 x 60.3 mm, 1 part

Commit message: upadeted panel
Parts:
- added 12V: 12V pad, wirepad:1,6/0,8
- added D1, D2, D3, D4, D5: BLUE, SparkFun-LED:LED-1206
- added GND: GND Pad, wirepad:1,6/0,8
- added R1, R2, R22, R3, R4: 330, rcl:R0805
Connections:
- new net 12V: 12V.1, R1.2, R2.2, R22.2, R3.2, R4.2
- new net GND: D1.C, D2.C, D3.C, D4.C, D5.C, GND.1
- new net N$1: D1.A, R22.1
- new net N$3: D2.A, R1.1
- new net N$5: D3.A, R2.1
- new net N$7: D4.A, R3.1
- new net N$9: D5.A, R4.1
Routing:
- net N$5: track 0.00 -> 83.8 mm
- net N$3: track 0.00 -> 81.6 mm
- net N$1: track 0.00 -> 72.3 mm
- net N$9: track 0.00 -> 49.3 mm
- net 12V: track 0.00 -> 38.6 mm
- net N$7: track 0.00 -> 27.4 mm
- net GND: track 0.00 -> 5.87 mm, vias 0 -> 5
- added copper zone on layer 1, net GND

Commit message: latest panel board using 'components'
Parts:
- added U$1, U$3: S_JACK_PANEL, GMSN-R2Project:S_JACK_PANEL
- added U$10, U$6, U$7, U$8, U$9: POT_PANEL, GMSN-R2Project:POT_PANEL
- added U$11: XLR_PANEL, GMSN-R2Project:XLR_PANEL
- added U$12, U$13, U$14, U$15: MOUNTING_HOLE, GMSN-R2Project:MOUNTING_HOLE
- added U$4, U$5: S_JACK_PANEL, GMSN-R2Project:S_JACK_PANEL@1
Routing:
- net GND: track 5.87 -> 26.3 mm, vias 5 -> 4
- net N$5: track 83.8 -> 96.5 mm
- net N$9: track 49.3 -> 46.2 mm
- removed copper zone on layer 1, net GND
Other:
- outline, holes or cut-outs redrawn
