File: PureRingMod.brd (EAGLE design)
At the start: 99 x 58.1 mm, 33 parts, among them IC1 TL074P, IC2 TL072P, X1 NC3FD-V

Commit message: updated BOM
Parts:
- D1: value (none) -> 1n4148
- D2: value (none) -> 1N4148
Changed lines of the file:
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@@
 <drawing>
 <settings>
-<setting alwaysvectorfont="yes"/>
+<setting alwaysvectorfont="no"/>
 <setting verticaltext="up"/>
 </settings>
@@
 <attribute name="NAME" x="6.9596" y="44.7802" size="1.27" layer="22" rot="MR180"/>
 </element>
-<element name="D1" library="adafruit" package="DO-1N4148" value="" x="83.82" y="26.67">
+<element name="D1" library="adafruit" package="DO-1N4148" value="1n4148" x="83.82" y="26.67">
 <attribute name="NAME" x="81.28" y="27.94" size="0.4064" layer="25"/>
 <attribute name="VALUE" x="81.788" y="26.416" size="0.6096" layer="21"/>
 </element>
-<element name="D2" library="adafruit" package="DO-1N4148" value="" x="83.82" y="30.48">
+<element name="D2" library="adafruit" package="DO-1N4148" value="1N4148" x="83.82" y="30.48">
 <attribute name="NAME" x="81.28" y="31.75" size="0.4064" layer="25"/>
 <attribute name="VALUE" x="81.788" y="30.226" size="0.6096" layer="21"/>
