File: PureRingMod-panel.sch (EAGLE design)
At the start: 0 parts

Commit message: upadeted panel
Parts:
- added 12V: 12V pad, wirepad:1,6/0,8
- added D1, D2, D3, D4, D5: BLUE, SparkFun-LED:LED-BLUE1206
- added GND: GND Pad, wirepad:1,6/0,8
- added R1, R2, R22, R3, R4: 330, rcl:R-US_R0805
Connections:
- new net 12V: 12V.P, R1.2, R2.2, R22.2, R3.2, R4.2
- new net GND: D1.C, D2.C, D3.C, D4.C, D5.C, GND.P
- new net N$1: D1.A, R22.1
- new net N$3: D2.A, R1.1
- new net N$5: D3.A, R2.1
- new net N$7: D4.A, R3.1
- new net N$9: D5.A, R4.1
Changed lines of the file:
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@@
 </classes>
 <parts>
+<part name="12V" library="wirepad" library_urn="urn:adsk.eagle:library:412" deviceset="1,6/0,8" device="" package3d_urn="urn:adsk.eagle:package:30830/1" value="12V pad"/>
+<part name="GND" library="wirepad" library_urn="urn:adsk.eagle:library:412" deviceset="1,6/0,8" device="" package3d_urn="urn:adsk.eagle:package:30830/1" value="GND Pad"/>
+<part name="R22" library="rcl" deviceset="R-US_" device="R0805" value="330"/>
+<part name="D1" library="SparkFun-LED" deviceset="LED-BLUE" device="1206" value="BLUE"/>
+<part name="R1" library="rcl" deviceset="R-US_" device="R0805" value="330"/>
+<part name="D2" library="SparkFun-LED" deviceset="LED-BLUE" device="1206" value="BLUE"/>
+<part name="R2" library="rcl" deviceset="R-US_" device="R0805" value="330"/>
+<part name="D3" library="SparkFun-LED" deviceset="LED-BLUE" device="1206" value="BLUE"/>
+<part name="R3" library="rcl" deviceset="R-US_" device="R0805" value="330"/>
+<part name="D4" library="SparkFun-LED" deviceset="LED-BLUE" device="1206" value="BLUE"/>
+<part name="R4" library="rcl" deviceset="R-US_" device="R0805" value="330"/>
+<part name="D5" library="SparkFun-LED" deviceset="LED-BLUE" device="1206" value="BLUE"/>
 </parts>
 <sheets>
@@
 </plain>
 <instances>
+<instance part="R22" gate="G$1" x="35.56" y="73.66" rot="R90">
+<attribute name="NAME" x="34.0614" y="69.85" size="1.778" layer="95" rot="R90"/>
+<attribute name="VALUE" x="38.862" y="69.85" size="1.778" layer="96" rot="R90"/>
+</instance>
+<instance part="D1" gate="G$1" x="35.56" y="60.96">
+<attribute name="NAME" x="32.131" y="56.388" size="1.778" layer="95" font="vector" rot="R90"/>
+<attribute name="VALUE" x="37.465" y="56.388" size="1.778" layer="96" font="vector" rot="R90" align="top-left"/>
+</instance>
+<instance part="R1" gate="G$1" x="45.72" y="73.66" rot="R90">
+<attribute name="NAME" x="44.2214" y="69.85" size="1.778" layer="95" rot="R90"/>
+<attribute name="VALUE" x="49.022" y="69.85" size="1.778" layer="96" rot="R90"/>
+</instance>
+<instance part="D2" gate="G$1" x="45.72" y="60.96">
+<attribute name="NAME" x="42.291" y="56.388" size="1.778" layer="95" font="vector" rot="R90"/>
+<attribute name="VALUE" x="47.625" y="56.388" size="1.778" layer="96" font="vector" rot="R90" align="top-left"/>
+</instance>
+<instance part="R2" gate="G$1" x="53.34" y="73.66" rot="R90">
+<attribute name="NAME" x="51.8414" y="69.85" size="1.778" layer="95" rot="R90"/>
+<attribute name="VALUE" x="56.642" y="69.85" size="1.778" layer="96" rot="R90"/>
+</instance>
+<instance part="D3" gate="G$1" x="53.34" y="60.96">
+<attribute name="NAME" x="49.911" y="56.388" size="1.778" layer="95" font="vector" rot="R90"/>
+<attribute name="VALUE" x="55.245" y="56.388" size="1.778" layer="96" font="vector" rot="R90" align="top-left"/>
+</instance>
+<instance part="R3" gate="G$1" x="60.96" y="73.66" rot="R90">
+<attribute name="NAME" x="59.4614" y="69.85" size="1.778" layer="95" rot="R90"/>
+<attribute name="VALUE" x="64.262" y="69.85" size="1.778" layer="96" rot="R90"/>
+</instance>
+<instance part="D4" gate="G$1" x="60.96" y="60.96">
+<attribute name="NAME" x="57.531" y="56.388" size="1.778" layer="95" font="vector" rot="R90"/>
+<attribute name="VALUE" x="62.865" y="56.388" size="1.778" layer="96" font="vector" rot="R90" align="top-left"/>
+</instance>
+<instance part="R4" gate="G$1" x="71.12" y="73.66" rot="R90">
+<attribute name="NAME" x="69.6214" y="69.85" size="1.778" layer="95" rot="R90"/>
+<attribute name="VALUE" x="74.422" y="69.85" size="1.778" layer="96" rot="R90"/>
+</instance>
+<instance part="D5" gate="G$1" x="71.12" y="60.96">
+<attribute name="NAME" x="67.691" y="56.388" size="1.778" layer="95" font="vector" rot="R90"/>
+<attribute name="VALUE" x="73.025" y="56.388" size="1.778" layer="96" font="vector" rot="R90" align="top-left"/>
+</instance>
 </instances>
 <busses>
 </busses>
 <nets>
+<net name="12V" class="0">
+<segment>
+<pinref part="R22" gate="G$1" pin="2"/>
+<wire x1="35.56" y1="78.74" x2="35.56" y2="81.28" width="0.1524" layer="91"/>
+<label x="35.56" y="81.28" size="1.778" layer="95" rot="R90" xref="yes"/>
+</segment>
+<segment>
+<pinref part="R1" gate="G$1" pin="2"/>
+<wire x1="45.72" y1="78.74" x2="45.72" y2="81.28" width="0.1524" layer="91"/>
+<label x="45.72" y="81.28" size="1.778" layer="95" rot="R90" xref="yes"/>
+</segment>
+<segment>
+<pinref part="R2" gate="G$1" pin="2"/>
+<wire x1="53.34" y1="78.74" x2="53.34" y2="81.28" width="0.1524" layer="91"/>
+<label x="53.34" y="81.28" size="1.778" layer="95" rot="R90" xref="yes"/>
+</segment>
+<segment>
+<pinref part="R3" gate="G$1" pin="2"/>
+<wire x1="60.96" y1="78.74" x2="60.96" y2="81.28" width="0.1524" layer="91"/>
+<label x="60.96" y="81.28" size="1.778" layer="95" rot="R90" xref="yes"/>
+</segment>
+<segment>
+<pinref part="R4" gate="G$1" pin="2"/>
+<wire x1="71.12" y1="78.74" x2="71.12" y2="81.28" width="0.1524" layer="91"/>
+<label x="71.12" y="81.28" size="1.778" layer="95" rot="R90" xref="yes"/>
+</segment>
+</net>
+<net name="N$1" class="0">
+<segment>
+<pinref part="R22" gate="G$1" pin="1"/>
+<pinref part="D1" gate="G$1" pin="A"/>
+<wire x1="35.56" y1="68.58" x2="35.56" y2="63.5" width="0.1524" layer="91"/>
+</segment>
+</net>
+<net name="N$3" class="0">
+<segment>
+<pinref part="R1" gate="G$1" pin="1"/>
+<pinref part="D2" gate="G$1" pin="A"/>
+<wire x1="45.72" y1="68.58" x2="45.72" y2="63.5" width="0.1524" layer="91"/>
+</segment>
+</net>
+<net name="GND" class="0">
+<segment>
+<wire x1="53.34" y1="55.88" x2="53.34" y2="45.72" width="0.1524" layer="91"/>
+<pinref part="D3" gate="G$1" pin="C"/>
+<pinref part="D1" gate="G$1" pin="C"/>
+<wire x1="35.56" y1="55.88" x2="35.56" y2="45.72" width="0.1524" layer="91"/>
+<wire x1="71.12" y1="55.88" x2="71.12" y2="45.72" width="0.1524" layer="91"/>
+<pinref part="D5" gate="G$1" pin="C"/>
+<wire x1="35.56" y1="45.72" x2="45.72" y2="45.72" width="0.1524" layer="91"/>
+<pinref part="D2" gate="G$1" pin="C"/>
+<wire x1="45.72" y1="45.72" x2="53.34" y2="45.72" width="0.1524" layer="91"/>
+<wire x1="53.34" y1="45.72" x2="60.96" y2="45.72" width="0.1524" layer="91"/>
+<wire x1="60.96" y1="45.72" x2="71.12" y2="45.72" width="0.1524" layer="91"/>
+<wire x1="45.72" y1="55.88" x2="45.72" y2="45.72" width="0.1524" layer="91"/>
+<junction x="45.72" y="45.72"/>
+<junction x="53.34" y="45.72"/>
+<pinref part="D4" gate="G$1" pin="C"/>
+<wire x1="60.96" y1="55.88" x2="60.96" y2="45.72" width="0.1524" layer="91"/>
+<junction x="60.96" y="45.72"/>
+<wire x1="53.34" y1="45.72" x2="53.34" y2="43.18" width="0.1524" layer="91"/>
+<label x="53.34" y="43.18" size="1.778" layer="95"/>
+</segment>
+</net>
+<net name="N$5" class="0">
+<segment>
+<pinref part="R2" gate="G$1" pin="1"/>
+<pinref part="D3" gate="G$1" pin="A"/>
+<wire x1="53.34" y1="68.58" x2="53.34" y2="63.5" width="0.1524" layer="91"/>
+</segment>
+</net>
+<net name="N$7" class="0">
+<segment>
+<pinref part="R3" gate="G$1" pin="1"/>
+<pinref part="D4" gate="G$1" pin="A"/>
+<wire x1="60.96" y1="68.58" x2="60.96" y2="63.5" width="0.1524" layer="91"/>
+</segment>
+</net>
+<net name="N$9" class="0">
+<segment>
+<pinref part="R4" gate="G$1" pin="1"/>
+<pinref part="D5" gate="G$1" pin="A"/>
+<wire x1="71.12" y1="68.58" x2="71.12" y2="63.5" width="0.1524" layer="91"/>
+</segment>
+</net>
 </nets>
 </sheet>
@@
 </plain>
 <instances>
+<instance part="12V" gate="P" x="22.86" y="68.58">
+<attribute name="NAME" x="21.717" y="70.4342" size="1.778" layer="95"/>
+<attribute name="VALUE" x="21.717" y="65.278" size="1.778" layer="96"/>
+</instance>
+<instance part="GND" gate="P" x="22.86" y="48.26">
+<attribute name="NAME" x="21.717" y="50.1142" size="1.778" layer="95"/>
+<attribute name="VALUE" x="21.717" y="44.958" size="1.778" layer="96"/>
+</instance>
 </instances>
 <busses>
 </busses>
 <nets>
+<net name="12V" class="0">
+<segment>
+<pinref part="12V" gate="P" pin="P"/>
+<wire x1="25.4" y1="68.58" x2="27.94" y2="68.58" width="0.1524" layer="91"/>
+<label x="27.94" y="68.58" size="1.778" layer="95"/>
+</segment>
+</net>
+<net name="GND" class="0">
+<segment>
+<pinref part="GND" gate="P" pin="P"/>
+<wire x1="25.4" y1="48.26" x2="27.94" y2="48.26" width="0.1524" layer="91"/>
+<label x="27.94" y="48.26" size="1.778" layer="95"/>
+</segment>
+</net>
 </nets>
 </sheet>
@@
 </schematic>
 </drawing>
+<compatibility>
+<note version="8.2" severity="warning">
+Since Version 8.2, EAGLE supports online libraries. The ids
+of those online libraries will not be understood (or retained)
+with this version.
+</note>
+<note version="8.3" severity="warning">
+Since Version 8.3, EAGLE supports URNs for individual library
+assets (packages, symbols, and devices). The URNs of those assets
+will not be understood (or retained) with this version.
+</note>
+<note version="8.3" severity="warning">
+Since Version 8.3, EAGLE supports the association of 3D packages
+with devices in libraries, schematics, and board files. Those 3D
+packages will not be understood (or retained) with this version.
+</note>
+</compatibility>
 </eagle>

Commit message: latest panel board using 'components'
Parts:
- added U$1, U$3: S_JACK_PANEL, GMSN-R2Project:S_JACK_PANEL
- added U$10, U$6, U$7, U$8, U$9: POT_PANEL, GMSN-R2Project:POT_PANEL
- added U$11: XLR_PANEL, GMSN-R2Project:XLR_PANEL
- added U$12, U$13, U$14, U$15: MOUNTING_HOLE, GMSN-R2Project:MOUNTING_HOLE
Changed lines of the file:
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@@
 <part name="R4" library="rcl" deviceset="R-US_" device="R0805" value="330"/>
 <part name="D5" library="SparkFun-LED" deviceset="LED-BLUE" device="1206" value="BLUE"/>
+<part name="U$1" library="GMSN-R2Project" deviceset="S_JACK_PANEL" device=""/>
+<part name="U$3" library="GMSN-R2Project" deviceset="S_JACK_PANEL" device=""/>
+<part name="U$6" library="GMSN-R2Project" deviceset="POT_PANEL" device=""/>
+<part name="U$7" library="GMSN-R2Project" deviceset="POT_PANEL" device=""/>
+<part name="U$8" library="GMSN-R2Project" deviceset="POT_PANEL" device=""/>
+<part name="U$9" library="GMSN-R2Project" deviceset="POT_PANEL" device=""/>
+<part name="U$10" library="GMSN-R2Project" deviceset="POT_PANEL" device=""/>
+<part name="U$12" library="GMSN-R2Project" deviceset="MOUNTING_HOLE" device=""/>
+<part name="U$13" library="GMSN-R2Project" deviceset="MOUNTING_HOLE" device=""/>
+<part name="U$14" library="GMSN-R2Project" deviceset="MOUNTING_HOLE" device=""/>
+<part name="U$15" library="GMSN-R2Project" deviceset="MOUNTING_HOLE" device=""/>
+<part name="U$11" library="GMSN-R2Project" deviceset="XLR_PANEL" device=""/>
 </parts>
 <sheets>
@@
 <attribute name="VALUE" x="73.025" y="56.388" size="1.778" layer="96" font="vector" rot="R90" align="top-left"/>
 </instance>
+<instance part="U$1" gate="G$1" x="7.62" y="96.52">
+<attribute name="NAME" x="5.08" y="100.584" size="1.778" layer="95"/>
+<attribute name="VALUE" x="5.08" y="90.424" size="1.778" layer="96"/>
+</instance>
+<instance part="U$3" gate="G$1" x="7.62" y="81.28">
+<attribute name="NAME" x="5.08" y="85.344" size="1.778" layer="95"/>
+<attribute name="VALUE" x="5.08" y="75.184" size="1.778" layer="96"/>
+</instance>
+<instance part="U$6" gate="G$1" x="7.62" y="63.5"/>
+<instance part="U$7" gate="G$1" x="7.62" y="53.34"/>
+<instance part="U$8" gate="G$1" x="7.62" y="45.72"/>
+<instance part="U$9" gate="G$1" x="7.62" y="38.1"/>
+<instance part="U$10" gate="G$1" x="7.62" y="27.94"/>
+<instance part="U$12" gate="G$1" x="88.9" y="91.44"/>
+<instance part="U$13" gate="G$1" x="88.9" y="81.28"/>
+<instance part="U$14" gate="G$1" x="88.9" y="73.66"/>
+<instance part="U$15" gate="G$1" x="88.9" y="60.96"/>
+<instance part="U$11" gate="G$1" x="88.9" y="45.72"/>
 </instances>
 <busses>
