File: V1.0/PureRingMod-panel.sch (EAGLE design)
At the start: 24 parts

Commit message: Panel layout and routing
Parts:
- removed 12V: 12V pad, wirepad:1,6/0,8
- removed D1, D2, D3, D4, D5: BLUE, SparkFun-LED:LED-BLUE1206
- removed GND: GND Pad, wirepad:1,6/0,8
- removed R1, R2, R22, R3, R4: 330, rcl:R-US_R0805
- removed U$1, U$3: S_JACK_PANEL, GMSN-R2Project:S_JACK_PANEL
- removed U$10, U$6, U$7, U$8, U$9: POT_PANEL, GMSN-R2Project:POT_PANEL
- removed U$11: XLR_PANEL, GMSN-R2Project:XLR_PANEL
- removed U$12, U$13, U$14, U$15: MOUNTING_HOLE, GMSN-R2Project:MOUNTING_HOLE
Connections:
- removed net 12V: 12V.P, R1.2, R2.2, R22.2, R3.2, R4.2
- removed net GND: D1.C, D2.C, D3.C, D4.C, D5.C, GND.P
- removed net N$1: D1.A, R22.1
- removed net N$3: D2.A, R1.1
- removed net N$5: D3.A, R2.1
- removed net N$7: D4.A, R3.1
- removed net N$9: D5.A, R4.1
